Commit message: edit urdf

File: resources/robots/ainex_description/urdf/ainex.urdf (robot description, URDF)
Before this commit: robot ainex, 28 links, 27 joints
Joints:
- joint l_sho_pitch: origin xyz=-5.4627E-05 0.052491 0.087448 rpy=-1 0 0 -> xyz=-5.4627E-05 0.052491 0.087448 rpy=0 0 0
- joint l_sho_roll: origin xyz=0.020003 0.021507 0 rpy=0 0 0 -> xyz=0.020003 0.021507 0 rpy=-1.57 0 0
- joint r_sho_pitch: origin xyz=-5.46273713767254E-05 -0.0524909514103703 0.0874480463620076 rpy=1 0 0 -> xyz=-5.46273713767254E-05 -0.0524909514103703 0.0874480463620076 rpy=0 0 0
- joint r_sho_roll: origin xyz=0.020003499818653 -0.021505961295104 0 rpy=0 0 0 -> xyz=0.020003499818653 -0.021505961295104 0 rpy=1.57 0 0
