Commit message: edit some parameters

File: resources/robots/ainex_description/meshes/ainex.urdf (robot description, URDF)
Before this commit: robot ainex, 28 links, 27 joints
Links:
- link l_ank_roll_link: geometry collision box size=0.12 0.08 0.004; visual box size=0.12 0.08 0.004
- link r_ank_roll_link: geometry collision box size=0.12 0.08 0.004; visual box size=0.12 0.08 0.004
Joints:
- joint head_pan: type fixed -> revolute
- joint head_tilt: type fixed -> revolute
- joint l_el_pitch: type fixed -> revolute
- joint l_el_yaw: type fixed -> revolute
- joint l_gripper: type fixed -> revolute
- joint l_sho_pitch: type fixed -> revolute
- joint l_sho_roll: origin xyz=0.020003 0.021507 0 rpy=-1.57 0 0 -> xyz=0.020003 0.021507 0 rpy=0 0 0; type fixed -> revolute
- joint r_el_pitch: type fixed -> revolute
- joint r_el_yaw: type fixed -> revolute
- joint r_gripper: type fixed -> revolute
- joint r_sho_pitch: type fixed -> revolute

File: resources/robots/ainex_description/urdf/ainex.urdf (robot description, URDF)
Before this commit: robot ainex, 28 links, 27 joints
Links:
- link l_ank_roll_link: geometry collision box size=0.12 0.08 0.004; visual box size=0.12 0.08 0.004
- link r_ank_roll_link: geometry collision box size=0.12 0.08 0.004; visual box size=0.12 0.08 0.004
